Commit message: modified urdf

File: gati_bot_model_description/urdf/lidar.urdf.xacro (robot description, xacro)
@@ -28,5 +28,5 @@
         <parent link="base_link" />
         <child link="laser_frame" />
-        <origin xyz="-0.045 0 ${base_height + 0.013}" rpy="0 0 0" />
+        <origin xyz="0.0 0 ${base_height + 0.013}" rpy="0 0 0" />
     </joint>
 </robot>

File: gati_bot_model_description/urdf/robot_model.urdf.xacro (robot description, xacro)
@@ -1,7 +1,7 @@
 <?xml version="1.0"?>
 <robot xmlns:xacro="http://www.ros.org/wiki/xacro">
-    <xacro:property name="base_length" value="0.138" />
-    <xacro:property name="base_width" value="0.133" />
-    <xacro:property name="base_height" value="0.120" />
+    <xacro:property name="base_length" value="0.140" />
+    <xacro:property name="base_width" value="0.160" />
+    <xacro:property name="base_height" value="0.170" />
     <xacro:property name="wheel_radius" value="0.0325" />
     <xacro:property name="wheel_length" value="0.025" />

Commit message: Added mesh files in urdf

File: gati_bot_model_description/urdf/lidar.urdf.xacro (robot description, xacro)
@@ -3,15 +3,15 @@
     <xacro:property name="laser_radius" value="0.035" />
     <xacro:property name="laser_height" value="0.023" />
-    <link name="laser_frame">
+    <link name="lidar_link">
         <visual>
             <geometry>
-                <cylinder radius="${laser_radius}" length="${laser_height}" />
+                <mesh filename="package://gati_bot_model_description/mesh/lidar.dae" scale="1 1 1"/>
             </geometry>
-            <origin xyz="0 0 0" rpy="0 0 0" />
+            <origin xyz="0.015 0 -0.035" rpy="1.5708 0 0" />
             <material name="black">
                 <color rgba="1 0 0 1" />
             </material>
         </visual>
-        <collision>
+        <!-- <collision>
             <geometry>
                 <cylinder radius="${laser_radius}" length="${laser_height}" />
@@ -22,11 +22,17 @@
             <origin xyz="0 0 0" rpy="0 0 0"/>
             <inertia ixx="0.000038" ixy="0" ixz="0" iyy="0.000038" iyz="0" izz="0.000061" />
-        </inertial>
+        </inertial> -->
     </link>
 <!-- x = -0.045 -->
-    <joint name="laser_joint" type="fixed">
+    <joint name="lidar_joint" type="fixed">
         <parent link="base_link" />
-        <child link="laser_frame" />
-        <origin xyz="0.0 0 ${base_height + 0.013}" rpy="0 0 0" />
+        <child link="lidar_link" />
+        <origin xyz="0.0 0 ${base_height + 0.031}" rpy="0 0 0" />
+    </joint>
+    <link name="laser_frame"></link>
+    <joint name="laser_frame_joint" type="fixed">
+        <parent link="lidar_link"/>
+        <child link="laser_frame"/>
+        <origin xyz="0 0 -0.01" rpy="0 0 0"/>
     </joint>
 </robot>

File: gati_bot_model_description/urdf/my_robot.urdf.xacro (robot description, xacro)
@@ -4,3 +4,4 @@
     <xacro:include filename="robot_model.urdf.xacro"/>
     <xacro:include filename="lidar.urdf.xacro"/>
+    <xacro:include filename="camera.urdf.xacro"/>
 </robot>

File: gati_bot_model_description/urdf/robot_model.urdf.xacro (robot description, xacro)
@@ -10,7 +10,8 @@
         <visual>
             <geometry>
-                <box size="${base_length} ${base_width} ${base_height}" />
+                <mesh filename="package://gati_bot_model_description/mesh/base.dae" scale="1 1 1"/>
+                <!--box size="${base_length} ${base_width} ${base_height}" /-->
             </geometry>
-            <origin xyz="0 0 ${base_height / 2.0}" rpy="0 0 0" />
+            <origin xyz="0 0 -0.016" rpy="1.5708 0 -1.5708" />
             <material name="Yellow" />
         </visual>
@@ -20,7 +21,8 @@
             <visual>
                 <geometry>
-                    <cylinder radius="${wheel_radius}" length="${wheel_length}" />
+                    <mesh filename="package://gati_bot_model_description/mesh/wheel_right.dae" scale="0.001 0.001 0.001"/>
+                    <!-- <cylinder radius="${wheel_radius}" length="${wheel_length}" /> -->
                 </geometry>
-                <origin xyz="0 0 0" rpy="${pi / 2.0} 0 0" />
+                <origin xyz="0 0.075 -0.0325" rpy="0 0 0" />
                 <material name="black" />
             </visual>
@@ -29,5 +31,5 @@
     <xacro:wheel_link prefix="right" />
     <xacro:wheel_link prefix="left" />
-    <link name="caster_wheel_link">
+    <!-- <link name="caster_wheel_link">
         <visual>
             <geometry>
@@ -37,14 +39,15 @@
             <material name="black" />
         </visual>
-    </link>
+    </link> -->
     <joint name="base_joint" type="fixed">
         <parent link="base_footprint" />
         <child link="base_link" />
-        <origin xyz="0 0 ${wheel_radius}" rpy="0 0 0"/>
+        <origin xyz="0 0 0" rpy="0 0 0"/>
     </joint>
     <joint name="base_right_wheel_joint" type="continuous">
         <parent link="base_link" />
         <child link="right_wheel_link" />
-        <origin xyz="-0.022 ${-(base_width + wheel_length) / 2.0} 0" rpy="0 0 0" />
+        <!-- <origin xyz="-0.022 ${-(base_width + wheel_length) / 2.0} 0" rpy="0 0 0" /> -->
+        <origin xyz="-0.0397 -0.0872 0.0289" rpy="0 0 0" />
         <axis xyz="0 1 0" />
     </joint>
@@ -52,11 +55,11 @@
         <parent link="base_link" />
         <child link="left_wheel_link" />
-        <origin xyz="-0.022 ${(base_width + wheel_length) / 2.0} 0" rpy="0 0 0" />
+        <origin xyz="-0.0397 0.0872 0.0289" rpy="3.1416 0 0" />
         <axis xyz="0 1 0" />
     </joint>
-    <joint name="base_caster_wheel_joint" type="fixed">
+    <!-- <joint name="base_caster_wheel_joint" type="fixed">
         <parent link="base_link" />
         <child link="caster_wheel_link" />
         <origin xyz="${base_length / 3.0} 0 ${-wheel_radius / 2.0}" rpy="0 0 0" />
-    </joint>
+    </joint> -->
 </robot>
